Commit message: fixed package name error

File: urdf/frame/dji_m100_frame.xacro (robot description, xacro)
@@ -2,5 +2,5 @@
 <robot xmlns:xacro="http://ros.org/wiki/xacro"
        name="dji_m100_frame" >
-  <xacro:include filename="$(find airsim_ros_wrapper)/urdf/materials.urdf.xacro" />
+  <xacro:include filename="$(find airsim_ros_client)/urdf/materials.urdf.xacro" />
   <xacro:property name="M_PI" value="3.1415926535897931" />
   <xacro:property name="base_mass" value="2.432" />
@@ -23,5 +23,5 @@
         <origin xyz="-0.35 -0.25 -0.14" rpy="${M_PI/2} 0 ${M_PI/2}" />
         <geometry>
-          <mesh filename="package://airsim_ros_wrapper/meshes/DJI_M100_CAD.STL" scale="0.001 0.001 0.001"/>
+          <mesh filename="package://airsim_ros_client/meshes/DJI_M100_CAD.STL" scale="0.001 0.001 0.001"/>
         </geometry>
         <material name="Black" />

File: urdf/robot/dji_m100_airsim.urdf (robot description, URDF)
Before this commit: robot dji_m100_airsim, 6 links, 5 joints
Links:
- link base_link: geometry collision cylinder length=0.218 radius=0.498; visual mesh filename=package://airsim_ros_client/meshes/DJI_M100_CAD.STL scale=0.001 0.001 0.001

File: urdf/robot/dji_m100_airsim.urdf.xacro (robot description, xacro)
@@ -2,6 +2,6 @@
 <robot xmlns:xacro="http://ros.org/wiki/xacro"
        name="dji_m100_airsim">
-   <xacro:include filename="$(find airsim_ros_wrapper)/urdf/frame/dji_m100_frame.xacro"/>
-   <xacro:include filename="$(find airsim_ros_wrapper)/urdf/sensors/airsim_cam.xacro"/>
+   <xacro:include filename="$(find airsim_ros_client)/urdf/frame/dji_m100_frame.xacro"/>
+   <xacro:include filename="$(find airsim_ros_client)/urdf/sensors/airsim_cam.xacro"/>
   <xacro:dji_m100_frame name="base"/>
   <xacro:airsim_cam name="base"/>
